File: hardware/publisher/publisher.kicad_pcb (KiCad board)
At the start: 2 copper layers, 78 x 57.5 mm, 32 parts, among them J1 Main Connector, J2 Main Debug, J3 uC Debug, J4 Reset Switch, J5 HV Select, J6 CTRL Select, Q1 BC337, Q2 BC337, Q3 BC337, U1 WeMos_D1_mini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

Commit message: upgraded sch and pcb to kicad 8
Other:
- net class Default removed
- net class Default Back removed
- net class Rail (up to 1A) removed
- net class Signals removed
- net class VBAT removed
